Commit message: chassis changed, fixed namespace issue with bridge

File: tuw_simulation/model/spike/body/chassis.xacro (robot description, xacro)
@@ -4,5 +4,5 @@
     <link name="base_link">
         <collision>
-            <origin xyz="0 0 0" rpy="0 0 0" />
+            <origin xyz="0 0 ${-wheel_z+wheel_radius}" rpy="0 0 0" />
             <geometry>
                 <box size="${base_length} ${base_width} ${base_height}" />
@@ -10,5 +10,5 @@
         </collision>
         <visual>
-            <origin xyz="0 0 0" rpy="0 0 0" />
+            <origin xyz="0 0 ${-wheel_z+wheel_radius}" rpy="0 0 0" />
             <geometry>
                 <box size="${base_length} ${base_width} ${base_height}" />
@@ -17,5 +17,5 @@
         </visual>
         <inertial>
-            <origin xyz="0 0 0" rpy="0 0 0" />
+            <origin xyz="0 0 ${-wheel_z+wheel_radius}" rpy="0 0 0" />
             <mass value="${base_mass}" />
             <!-- intertia for a box -->
@@ -31,5 +31,5 @@
         <parent link="base_link"/>
         <child link="base_footprint"/>
-        <origin xyz="0.0 0.0 ${-(wheel_radius+wheel_offset)}" rpy="0 0 0"/>
+        <origin xyz="0.0 0.0 ${-wheel_z+wheel_radius}" rpy="0 0 0"/>
     </joint>
 </robot>

File: tuw_simulation/model/spike/body/properties.xacro (robot description, xacro)
@@ -2,5 +2,5 @@
 <robot xmlns:xacro="http://ros.org/wiki/xacro">
     <xacro:property name="PI" value="3.1415926535897931" />
-    <xacro:property name="base_mass" value="1.5" />
+    <!-- <xacro:property name="base_mass" value="1.5" />
     <xacro:property name="base_width" value="0.31"/>
     <xacro:property name="base_length" value="0.42"/>
@@ -12,4 +12,26 @@
     <xacro:property name="wheel_xoff" value="0.12"/>
     <xacro:property name="wheel_ygap" value="0.025"/>
-    <xacro:property name="caster_xoff" value="0.14"/>
+    <xacro:property name="caster_xoff" value="0.14"/> -->
+    <!-- x nach vorne | y breite | z höhe -->
+    <!-- wheel -->
+    <xacro:property name="wheel_x" value="-0.07874"/>
+    <xacro:property name="wheel_z" value="-0.015748"/>
+    <xacro:property name="wheel_y" value="0.055118"/>
+    <xacro:property name="wheel_diameter" value="0.055"/> <!-- lego diameter 56mm -->
+    <xacro:property name="wheel_radius" value="${wheel_diameter/2}"/>
+    <xacro:property name="wheel_len" value="0.0137"/> <!-- lego len 14mm -->
+    <xacro:property name="wheel_mass" value="0.1"/> <!-- kein gewicht von lego noch abwiegen-->
+    <!-- Caster wheel -->
+    <xacro:property name="caster_z" value="-0.033858"/>
+    <xacro:property name="caster_x" value="0.05512"/>
+    <xacro:property name="caster_y" value="0"/>
+    <xacro:property name="caster_diameter" value="0.0188"/>
+    <xacro:property name="caster_radius" value="${caster_diameter/2}"/>
+    <xacro:property name="caster_mass" value="0.05"/>
+    <!-- base Chassis -->
+    <!-- Werte sind nur vorrübergehend -->
+    <xacro:property name="base_mass" value="0.7"/>
+    <xacro:property name="base_width" value="${wheel_y * 2}"/>
+    <xacro:property name="base_length" value="0.170"/>
+    <xacro:property name="base_height" value="0.09"/>
 </robot>

File: tuw_simulation/model/spike/body/wheels.xacro (robot description, xacro)
@@ -2,13 +2,11 @@
 <robot xmlns:xacro="http://ros.org/wiki/xacro">
     <!-- Wheel Macro -->
-    <xacro:macro name="wheel" params="prefix x_reflect y_reflect">
+    <xacro:macro name="wheel" params="prefix y_reflect">
         <!-- Wheel Joint -->
         <joint name="${prefix}_wheel_joint" type="continuous">
             <parent link="base_link" />
             <child link="${prefix}_wheel" />
-            <origin xyz="${x_reflect*wheel_offset} ${y_reflect*(base_width/2+wheel_ygap)} ${-wheel_offset}" rpy="0 0 0" />
+            <origin xyz="${wheel_x} ${y_reflect*wheel_y} ${wheel_z}" rpy="0 0 0" />
             <axis xyz="0 1 0" />
-            <dynamics damping="0.2" />
-            <limit effort="100" velocity="3.0" />
         </joint>
         <!-- Wheel Link -->
@@ -36,13 +34,25 @@
                     ixy="0.0" ixz="0.0" iyz="0.0" />
             </inertial>
+            <gazebo reference="${prefix}_wheel">
+                <mu1 value="10.0"/>
+                <mu2 value="10.0"/>
+                <kp value="10000000.0"/>
+                <kd value="1.0"/>
+                <fdir1 value="1 1 0"/>
+            </gazebo>
         </link>
     </xacro:macro>
-    <xacro:wheel prefix="left" x_reflect="-1" y_reflect="1" />
-    <xacro:wheel prefix="right" x_reflect="-1" y_reflect="-1" />
+    <xacro:wheel prefix="left" y_reflect="1" />
+    <xacro:wheel prefix="right" y_reflect="-1" />
+    <joint name="caster_joint_gz" type="continuous">
+        <parent link="base_link"/>
+        <child link="front_caster_gz"/>
+        <origin xyz="${caster_x} ${caster_y} ${caster_z}" rpy="0 0 0"/>
+    </joint>
     <!-- Caster Wheel -->
-    <link name="front_caster">
+    <link name="front_caster_gz">
         <visual>
             <geometry>
-                <sphere radius="${(wheel_radius+wheel_offset-(base_height/2))}"/>
+                <sphere radius="${caster_radius}"/>
             </geometry>
             <material name="black"/>
@@ -50,12 +60,23 @@
         <collision>
             <geometry>
-                <sphere radius="${(wheel_radius+wheel_offset-(base_height/2))}"/>
+                <sphere radius="${caster_radius}"/>
             </geometry>
         </collision>
+        <inertial>
+            <origin xyz="0 0 0" rpy="0 0 0" />
+            <mass value="${caster_mass}" />
+            <inertia
+                ixx="${2/5 * caster_mass * caster_radius*caster_radius}"
+                iyy="${2/5 * caster_mass * caster_radius*caster_radius}"
+                izz="${2/5 * caster_mass * caster_radius*caster_radius}"
+                ixy="0.0" ixz="0.0" iyz="0.0" />
+        </inertial>
+        <gazebo reference="front_caster_gz">
+            <mu1 value="0.0"/>
+            <mu2 value="0.0"/>
+            <kp value="10000000.0"/>
+            <kd value="1.0"/>
+            <fdir1 value="1 0 0"/>
+        </gazebo>
     </link>
-    <joint name="caster_joint" type="fixed">
-        <parent link="base_link"/>
-        <child link="front_caster"/>
-        <origin xyz="${caster_xoff} 0.0 ${-(base_height/2)}" rpy="0 0 0"/>
-    </joint>
 </robot>
