Commit message: added camera

File: tuw_simulation/model/spike/body/body.xacro (robot description, xacro)
@@ -9,3 +9,4 @@
     <!-- include wheels -->
     <xacro:include filename="wheels.xacro"/>
+    <xacro:include filename="camera.xacro"/>
 </robot>

File: tuw_simulation/model/spike/body/properties.xacro (robot description, xacro)
@@ -35,3 +35,8 @@
     <xacro:property name="base_length" value="0.170"/>
     <xacro:property name="base_height" value="0.09"/>
+    <!-- camera -->
+    <xacro:property name="camera_x" value="0.09167"/>
+    <xacro:property name="camera_y" value="0.0"/>
+    <xacro:property name="camera_z" value="0.06464"/>
+    <xacro:property name="camera_angle" value="24.74"/>
 </robot>

Commit message: ray_localizer: calculate rays in image space

File: tuw_simulation/model/spike/body/body.xacro (robot description, xacro)
@@ -10,3 +10,4 @@
     <xacro:include filename="wheels.xacro"/>
     <xacro:include filename="camera.xacro"/>
+    <xacro:include filename="ray_frame.xacro"/>
 </robot>

File: tuw_simulation/model/spike/body/properties.xacro (robot description, xacro)
@@ -40,3 +40,4 @@
     <xacro:property name="camera_z" value="0.06464"/>
     <xacro:property name="camera_angle" value="24.74"/>
+    <xacro:property name="ray_origin_offset" value="0.15"/>
 </robot>
