Commit message: added inertias

File: tuw_description/model/spike/body/camera.xacro (robot description, xacro)
@@ -12,8 +12,18 @@
             <origin xyz="0 0 0" rpy="0 0 0"/>
             <geometry>
-                <box size="0.005 0.025 0.025"/>
+                <box size="${camera_width} ${camera_length} ${camera_height}"/>
             </geometry>
             <material name="green"/>
         </visual>
+        <inertial>
+            <origin xyz="0 0 0" rpy="0 0 0" />
+            <mass value="${camera_mass}" />
+            <!-- intertia for a box -->
+            <inertia
+                ixx="${camera_mass / 12.0 * (camera_length*camera_length + camera_height*camera_height)}"
+                iyy="${camera_mass / 12.0 * (camera_height*camera_height + camera_width*camera_width)}"
+                izz="${camera_mass / 12.0 * (camera_width*camera_width + camera_length*camera_length)}"
+                ixy="0.0" ixz="0.0" iyz="0.0" />
+        </inertial>
     </link>
     <link name="camera_optical"/>

File: tuw_description/model/spike/body/chassis.xacro (robot description, xacro)
@@ -1,4 +1,16 @@
 <?xml version="1.0"?>
 <robot xmlns:xacro="http://ros.org/wiki/xacro">
+    <xacro:macro name="engine_inertia" params="y_reflect">
+        <inertial>
+            <origin xyz="${engine_x} ${engine_y} ${engine_z}" rpy="0 0 0" />
+            <mass value="${engine_mass}" />
+            <!-- intertia for a box -->
+            <inertia
+                ixx="${engine_mass / 12.0 * (engine_length*engine_length + engine_height*engine_height)}"
+                iyy="${engine_mass / 12.0 * (engine_height*engine_height + engine_width*engine_width)}"
+                izz="${engine_mass / 12.0 * (engine_width*engine_width + engine_length*engine_length)}"
+                ixy="0.0" ixz="0.0" iyz="0.0" />
+        </inertial>
+    </xacro:macro>
     <!-- Base Link (Chassis) -->
     <link name="base_link">
@@ -12,18 +24,52 @@
             <origin xyz="0 0 ${-wheel_z+wheel_radius}" rpy="0 0 0" />
             <geometry>
-                <box size="${base_length} ${base_width} ${base_height}" />
+                <box size="${base_length/10} ${base_width/10} ${base_height/10}" />
             </geometry>
             <material name="orange" />
         </visual>
         <inertial>
-            <origin xyz="0 0 ${-wheel_z+wheel_radius}" rpy="0 0 0" />
-            <mass value="${base_mass}" />
+            <origin xyz="0.02317682 0.00000690 0.01649155"/>
+            <mass value="${chassis_mass}"/>
+            <inertia ixx="0.00019830" ixy="-0.00000003" ixz="-0.00004422" iyy="0.00034369" iyz="-0.00000001" izz="0.00033507"/>
+        </inertial>
+        <!-- battery -->
+        <visual>
+            <origin xyz="${battery_x} ${battery_y} ${battery_z}" rpy="0 0 ${pi/2}" />
+            <geometry>
+                <box size="${battery_length} ${battery_width} ${battery_height}" />
+            </geometry>
+            <material name="black" />
+        </visual>
+        <inertial>
+            <origin xyz="${battery_x} ${battery_y} ${battery_z}" rpy="0 0 ${pi/2}" />
+            <mass value="${battery_mass}" />
             <!-- intertia for a box -->
             <inertia
-                ixx="${base_mass / 12.0 * (base_length*base_length + base_height*base_height)}"
-                iyy="${base_mass / 12.0 * (base_height*base_height + base_width*base_width)}"
-                izz="${base_mass / 12.0 * (base_width*base_width + base_length*base_length)}"
+                ixx="${battery_mass / 12.0 * (battery_length*battery_length + battery_height*battery_height)}"
+                iyy="${battery_mass / 12.0 * (battery_height*battery_height + battery_width*battery_width)}"
+                izz="${battery_mass / 12.0 * (battery_width*battery_width + battery_length*battery_length)}"
                 ixy="0.0" ixz="0.0" iyz="0.0" />
         </inertial>
+        <!-- PI -->
+        <visual>
+            <origin xyz="${pi_x} ${pi_y} ${pi_z}" rpy="0 0 ${pi/2}" />
+            <geometry>
+                <box size="${pi_length} ${pi_width} ${pi_height}" />
+            </geometry>
+            <material name="black" />
+        </visual>
+        <inertial>
+            <origin xyz="${pi_x} ${pi_y} ${pi_z}" rpy="0 0 ${pi/2}" />
+            <mass value="${pi_mass}" />
+            <!-- intertia for a box -->
+            <inertia
+                ixx="${pi_mass / 12.0 * (pi_length*pi_length + pi_height*pi_height)}"
+                iyy="${pi_mass / 12.0 * (pi_height*pi_height + pi_width*pi_width)}"
+                izz="${pi_mass / 12.0 * (pi_width*pi_width + pi_length*pi_length)}"
+                ixy="0.0" ixz="0.0" iyz="0.0" />
+        </inertial>
+        <!-- engine -->
+        <xacro:engine_inertia y_reflect="1" />
+        <xacro:engine_inertia y_reflect="-1" />
     </link>
     <link name="base_footprint"/>

File: tuw_description/model/spike/body/properties.xacro (robot description, xacro)
@@ -2,5 +2,5 @@
 <robot xmlns:xacro="http://ros.org/wiki/xacro">
     <xacro:property name="PI" value="3.1415926535897931" />
-    <!-- wheel -->
+    <!-- wheel from blender -->
     <xacro:property name="wheel_x" value="-0.08"/>
     <xacro:property name="wheel_z" value="-0.016"/>
@@ -9,6 +9,6 @@
     <xacro:property name="wheel_radius" value="${wheel_diameter/2}"/>
     <xacro:property name="wheel_len" value="0.0139"/> <!-- lego len 14mm -->
-    <xacro:property name="wheel_mass" value="0.1"/> <!-- kein gewicht von lego noch abwiegen-->
-    <!-- Caster wheel -->
+    <xacro:property name="wheel_mass" value="0.016"/> <!-- kein gewicht von lego noch abwiegen-->
+    <!-- Caster wheel from blender -->
     <xacro:property name="caster_z" value="-0.0344"/>
     <xacro:property name="caster_x" value="0.056002"/>
@@ -19,26 +19,40 @@
     <!-- base Chassis -->
     <!-- Werte sind nur vorrübergehend -->
-    <xacro:property name="base_mass" value="0.7"/>
+    <xacro:property name="chassis_mass" value="0.123"/>
     <xacro:property name="base_width" value="${wheel_y * 2}"/>
     <xacro:property name="base_length" value="0.170"/>
     <xacro:property name="base_height" value="0.09"/>
-    <!-- camera -->
+    <!-- from blender -->
     <xacro:property name="camera_x" value="0.099737"/>
     <xacro:property name="camera_y" value="0.0"/>
     <xacro:property name="camera_z" value="0.065674"/>
     <xacro:property name="camera_angle" value="24.737"/>
+    <xacro:property name="camera_width" value="0.005"/>
+    <xacro:property name="camera_length" value="0.025"/>
+    <xacro:property name="camera_height" value="0.025"/>
+    <xacro:property name="camera_mass" value="0.02"/>
+    <!-- from cad / blender -->
     <xacro:property name="battery_width" value="0.041"/>
     <xacro:property name="battery_length" value="0.071"/>
     <xacro:property name="battery_height" value="0.022"/>
-    <xacro:property name="battery_x" value="0.012"/>
+    <xacro:property name="battery_x" value="0.016"/>
     <xacro:property name="battery_y" value="0.0"/>
     <xacro:property name="battery_z" value="${-0.004 - (battery_height/2)}"/>
-    <xacro:property name="battery_weight" value="0.0"/>
+    <xacro:property name="battery_mass" value="0.150"/>
+    <!-- from cad / blender -->
     <xacro:property name="pi_width" value="0.056"/>
     <xacro:property name="pi_length" value="0.087"/>
     <xacro:property name="pi_height" value="0.020"/>
-    <xacro:property name="pi_x" value="24.74"/>
-    <xacro:property name="pi_y" value="24.74"/>
-    <xacro:property name="pi_z" value="24.74"/>
-    <xacro:property name="pi_weight" value="0.0"/>
+    <xacro:property name="pi_x" value="0.016"/>
+    <xacro:property name="pi_y" value="0.0"/>
+    <xacro:property name="pi_z" value="${+0.004 + pi_height/2}"/>
+    <xacro:property name="pi_mass" value="0.100"/>
+    <!-- from blender  -->
+    <xacro:property name="engine_width" value="0.024"/>
+    <xacro:property name="engine_length" value="0.0715"/>
+    <xacro:property name="engine_height" value="0.024"/>
+    <xacro:property name="engine_x" value="-0.056"/>
+    <xacro:property name="engine_y" value="0.032"/>
+    <xacro:property name="engine_z" value="${-0.004 - engine_height/2}"/>
+    <xacro:property name="engine_mass" value="0.045"/>
 </robot>
