Commit message: added extra links for inertia added ray_frame

File: tuw_description/model/spike/body/body.xacro (robot description, xacro)
@@ -9,4 +9,12 @@
     <!-- include wheels -->
     <xacro:include filename="wheels.xacro"/>
+    <!-- include pi -->
+    <xacro:include filename="pi.xacro"/>
+    <!-- include battery -->
+    <xacro:include filename="battery.xacro"/>
+    <!-- include engines -->
+    <xacro:include filename="engine.xacro"/>
+    <!-- include camera -->
     <xacro:include filename="camera.xacro"/>
+    <xacro:include filename="ray_frame.xacro"/>
 </robot>

File: tuw_description/model/spike/body/camera.xacro (robot description, xacro)
@@ -12,5 +12,5 @@
             <origin xyz="0 0 0" rpy="0 0 0"/>
             <geometry>
-                <box size="${camera_width} ${camera_length} ${camera_height}"/>
+                <box size="${camera_length} ${camera_width} ${camera_height}"/>
             </geometry>
             <material name="green"/>

File: tuw_description/model/spike/body/chassis.xacro (robot description, xacro)
@@ -1,20 +1,8 @@
 <?xml version="1.0"?>
 <robot xmlns:xacro="http://ros.org/wiki/xacro">
-    <xacro:macro name="engine_inertia" params="y_reflect">
-        <inertial>
-            <origin xyz="${engine_x} ${engine_y} ${engine_z}" rpy="0 0 0" />
-            <mass value="${engine_mass}" />
-            <!-- intertia for a box -->
-            <inertia
-                ixx="${engine_mass / 12.0 * (engine_length*engine_length + engine_height*engine_height)}"
-                iyy="${engine_mass / 12.0 * (engine_height*engine_height + engine_width*engine_width)}"
-                izz="${engine_mass / 12.0 * (engine_width*engine_width + engine_length*engine_length)}"
-                ixy="0.0" ixz="0.0" iyz="0.0" />
-        </inertial>
-    </xacro:macro>
     <!-- Base Link (Chassis) -->
     <link name="base_link">
         <collision>
-            <origin xyz="0 0 ${-wheel_z+wheel_radius}" rpy="0 0 0" />
+            <origin xyz="0 0 ${base_height/2}" rpy="0 0 0" />
             <geometry>
                 <box size="${base_length} ${base_width} ${base_height}" />
@@ -22,5 +10,5 @@
         </collision>
         <visual>
-            <origin xyz="0 0 ${-wheel_z+wheel_radius}" rpy="0 0 0" />
+            <origin xyz="0 0 ${base_height/2}" rpy="0 0 0" />
             <geometry>
                 <box size="${base_length/10} ${base_width/10} ${base_height/10}" />
@@ -28,48 +16,13 @@
             <material name="orange" />
         </visual>
-        <inertial>
-            <origin xyz="0.02317682 0.00000690 0.01649155"/>
-            <mass value="${chassis_mass}"/>
-            <inertia ixx="0.00019830" ixy="-0.00000003" ixz="-0.00004422" iyy="0.00034369" iyz="-0.00000001" izz="0.00033507"/>
-        </inertial>
-        <!-- battery -->
-        <visual>
-            <origin xyz="${battery_x} ${battery_y} ${battery_z}" rpy="0 0 ${pi/2}" />
-            <geometry>
-                <box size="${battery_length} ${battery_width} ${battery_height}" />
-            </geometry>
-            <material name="black" />
-        </visual>
-        <inertial>
-            <origin xyz="${battery_x} ${battery_y} ${battery_z}" rpy="0 0 ${pi/2}" />
-            <mass value="${battery_mass}" />
-            <!-- intertia for a box -->
+        <inertial name="base_link_inertia">
+            <origin xyz="0 0 ${base_height/2}" rpy="0 0 0" />
+            <mass value="${chassis_mass}" />
             <inertia
-                ixx="${battery_mass / 12.0 * (battery_length*battery_length + battery_height*battery_height)}"
-                iyy="${battery_mass / 12.0 * (battery_height*battery_height + battery_width*battery_width)}"
-                izz="${battery_mass / 12.0 * (battery_width*battery_width + battery_length*battery_length)}"
+                ixx="${chassis_mass / 12.0 * (base_length*base_length + base_height*base_height)}"
+                iyy="${chassis_mass / 12.0 * (base_height*base_height + base_width*base_width)}"
+                izz="${chassis_mass / 12.0 * (base_width*base_width + base_length*base_length)}"
                 ixy="0.0" ixz="0.0" iyz="0.0" />
         </inertial>
-        <!-- PI -->
-        <visual>
-            <origin xyz="${pi_x} ${pi_y} ${pi_z}" rpy="0 0 ${pi/2}" />
-            <geometry>
-                <box size="${pi_length} ${pi_width} ${pi_height}" />
-            </geometry>
-            <material name="black" />
-        </visual>
-        <inertial>
-            <origin xyz="${pi_x} ${pi_y} ${pi_z}" rpy="0 0 ${pi/2}" />
-            <mass value="${pi_mass}" />
-            <!-- intertia for a box -->
-            <inertia
-                ixx="${pi_mass / 12.0 * (pi_length*pi_length + pi_height*pi_height)}"
-                iyy="${pi_mass / 12.0 * (pi_height*pi_height + pi_width*pi_width)}"
-                izz="${pi_mass / 12.0 * (pi_width*pi_width + pi_length*pi_length)}"
-                ixy="0.0" ixz="0.0" iyz="0.0" />
-        </inertial>
-        <!-- engine -->
-        <xacro:engine_inertia y_reflect="1" />
-        <xacro:engine_inertia y_reflect="-1" />
     </link>
     <link name="base_footprint"/>
@@ -77,5 +30,5 @@
         <parent link="base_link"/>
         <child link="base_footprint"/>
-        <origin xyz="0.0 0.0 ${-wheel_z+wheel_radius}" rpy="0 0 0"/>
+        <origin xyz="0.0 0.0 ${wheel_z-wheel_radius}" rpy="0 0 0"/>
     </joint>
 </robot>

File: tuw_description/model/spike/body/properties.xacro (robot description, xacro)
@@ -16,11 +16,11 @@
     <xacro:property name="caster_diameter" value="0.0188"/>
     <xacro:property name="caster_radius" value="${caster_diameter/2}"/>
-    <xacro:property name="caster_mass" value="0.05"/>
+    <xacro:property name="caster_mass" value="0.005"/>
     <!-- base Chassis -->
     <!-- Werte sind nur vorrübergehend -->
     <xacro:property name="chassis_mass" value="0.123"/>
-    <xacro:property name="base_width" value="${wheel_y * 2}"/>
+    <xacro:property name="base_width" value="0.0879"/>
     <xacro:property name="base_length" value="0.170"/>
-    <xacro:property name="base_height" value="0.09"/>
+    <xacro:property name="base_height" value="0.064"/>
     <!-- from blender -->
     <xacro:property name="camera_x" value="0.099737"/>
@@ -28,6 +28,6 @@
     <xacro:property name="camera_z" value="0.065674"/>
     <xacro:property name="camera_angle" value="24.737"/>
-    <xacro:property name="camera_width" value="0.005"/>
-    <xacro:property name="camera_length" value="0.025"/>
+    <xacro:property name="camera_width" value="0.025"/>
+    <xacro:property name="camera_length" value="0.005"/>
     <xacro:property name="camera_height" value="0.025"/>
     <xacro:property name="camera_mass" value="0.02"/>
@@ -56,3 +56,4 @@
     <xacro:property name="engine_z" value="${-0.004 - engine_height/2}"/>
     <xacro:property name="engine_mass" value="0.045"/>
+    <xacro:property name="ray_origin_offset" value="0.15"/>
 </robot>

File: tuw_description/model/spike/body/wheels.xacro (robot description, xacro)
@@ -34,16 +34,9 @@
                     ixy="0.0" ixz="0.0" iyz="0.0" />
             </inertial>
-            <gazebo reference="${prefix}_wheel">
-                <mu1 value="10.0"/>
-                <mu2 value="10.0"/>
-                <kp value="10000000.0"/>
-                <kd value="1.0"/>
-                <fdir1 value="1 1 0"/>
-            </gazebo>
         </link>
     </xacro:macro>
     <xacro:wheel prefix="left" y_reflect="1" />
     <xacro:wheel prefix="right" y_reflect="-1" />
-    <joint name="caster_joint_gz" type="continuous">
+    <joint name="caster_joint_gz" type="fixed">
         <parent link="base_link"/>
         <child link="front_caster_gz"/>
@@ -72,11 +65,11 @@
                 ixy="0.0" ixz="0.0" iyz="0.0" />
         </inertial>
-        <gazebo reference="front_caster_gz">
-            <mu1 value="0.0"/>
-            <mu2 value="0.0"/>
-            <kp value="10000000.0"/>
-            <kd value="1.0"/>
-            <fdir1 value="1 0 0"/>
-        </gazebo>
     </link>
+    <gazebo reference="front_caster_gz">
+        <mu1 value="0.0"/>
+        <mu2 value="0.0"/>
+        <kp value="10000000.0"/>
+        <kd value="1.0"/>
+        <fdir1 value="1 0 0"/>
+    </gazebo>
 </robot>
