Commit message: deleted engine visual

File: tuw_description/model/spike/body/engine.xacro (robot description, xacro)
@@ -10,11 +10,4 @@
         </joint>
         <link name="engine_${prefix}">
-            <visual>
-                <origin xyz="0 0 0" rpy="0 0 0" />
-                <geometry>
-                    <box size="${engine_length} ${engine_width} ${engine_height}" />
-                </geometry>
-                <material name="black" />
-            </visual>
             <inertial>
                 <origin xyz="0 0 0" rpy="0 0 0" />
