Commit message: tuw_spike_camera: get amcl to work

File: tuw_description/model/spike/body/chassis.xacro (robot description, xacro)
@@ -26,9 +26,15 @@
         </inertial>
     </link>
+    <link name="base_odom"/>
     <link name="base_footprint"/>
+    <joint name="odom_joint" type="fixed">
+        <parent link="base_odom"/>
+        <child link="base_footprint"/>
+        <origin xyz="${-wheel_x} 0.0 0.0" rpy="0 0 0"/>
+    </joint>
     <joint name="base_joint" type="fixed">
-        <parent link="base_link"/>
-        <child link="base_footprint"/>
-        <origin xyz="0.0 0.0 ${wheel_z-wheel_radius}" rpy="0 0 0"/>
+        <parent link="base_footprint"/>
+        <child link="base_link"/>
+        <origin xyz="0.0 0.0 ${-wheel_z+wheel_radius}" rpy="0 0 0"/>
     </joint>
 </robot>

File: tuw_description/model/spike/body/plugins.xacro (robot description, xacro)
@@ -12,8 +12,8 @@
             <left_joint>left_wheel_joint</left_joint>
             <right_joint>right_wheel_joint</right_joint>
-            <wheel_separation>${base_width}</wheel_separation>
+            <wheel_separation>${2 * wheel_y + wheel_len}</wheel_separation>
             <wheel_radius>${wheel_radius}</wheel_radius>
             <frame_id>odom</frame_id>
-            <child_frame_id>base_link</child_frame_id>
+            <child_frame_id>base_odom</child_frame_id>
             <odom_publish_frequency>10</odom_publish_frequency>
             <!-- output -->

File: tuw_description/model/spike/body/wheels.xacro (robot description, xacro)
@@ -35,4 +35,11 @@
             </inertial>
         </link>
+        <gazebo reference="${prefix}_wheel">
+            <mu1 value="1.0"/>
+            <mu2 value="1.0"/>
+            <kp value="10000000.0"/>
+            <kd value="1.0"/>
+            <fdir1 value="1 0 0"/>
+        </gazebo>
     </xacro:macro>
     <xacro:wheel prefix="left" y_reflect="1" />
