Commit message: added record node

File: tuw_description/model/spike/body/wheels.xacro (robot description, xacro)
@@ -8,5 +8,7 @@
             <child link="${prefix}_wheel" />
             <origin xyz="${wheel_x} ${y_reflect*wheel_y} ${wheel_z}" rpy="0 0 0" />
-            <axis xyz="0 1 0" />
+            <axis xyz="0 1 0"/>
+            <!-- <dynamics damping="0.2" />
+            <limit effort="100" velocity="3.0" /> -->
         </joint>
         <!-- Wheel Link -->
@@ -69,6 +71,4 @@
         <mu1 value="0.0"/>
         <mu2 value="0.0"/>
-        <kp value="10000000.0"/>
-        <kd value="1.0"/>
         <fdir1 value="1 0 0"/>
     </gazebo>
