Commit message: clean up robot description, added model to simulation

File: tuw_spike_description/model/spike/body/battery.xacro (robot description, xacro)
@@ -14,5 +14,5 @@
                 <box size="${battery_length} ${battery_width} ${battery_height}" />
             </geometry>
-            <material name="black" />
+            <material name="grey" />
         </visual>
         <inertial name="battery_inertia">

File: tuw_spike_description/model/spike/body/chassis.xacro (robot description, xacro)
@@ -4,5 +4,5 @@
     <link name="base_link">
         <collision>
-            <origin xyz="0 0 ${base_height/2}" rpy="0 0 0" />
+            <origin xyz="0 0 0" rpy="0 0 0" />
             <geometry>
                 <box size="${base_length} ${base_width} ${base_height}" />
@@ -10,7 +10,8 @@
         </collision>
         <visual>
-            <origin xyz="0 0 ${base_height/2}" rpy="0 0 0" />
+            <origin xyz="0 0 0" rpy="0 0 0" />
             <geometry>
-                <box size="${base_length/10} ${base_width/10} ${base_height/10}" />
+                <box size="${base_length} ${base_width} ${base_height}" />
+                 <!-- <mesh filename="package://tuw_spike_description/model/spike/body/mesh/model_chassis.dae"/> -->
             </geometry>
             <material name="orange" />

File: tuw_spike_description/model/spike/body/materials.xacro (robot description, xacro)
@@ -4,7 +4,4 @@
     <color rgba="0.0 0.0 0.0 1.0"/>
   </material>
-  <!-- <material name="blue">
-    <color rgba="0.0 0.0 0.8 1.0"/>
-  </material> -->
   <material name="green">
     <color rgba="0.0 0.8 0.0 1.0"/>

File: tuw_spike_description/model/spike/body/pi.xacro (robot description, xacro)
@@ -14,5 +14,5 @@
                 <box size="${pi_length} ${pi_width} ${pi_height}" />
             </geometry>
-            <material name="black" />
+            <material name="grey" />
         </visual>
         <inertial name="pi_inertia">

File: tuw_spike_description/model/spike/body/plugins.xacro (robot description, xacro)
@@ -22,10 +22,10 @@
             <tf_topic>${namespace}/tf</tf_topic>
             <!-- limits -->
-            <min_linear_velocity>-0.95</min_linear_velocity>
-            <max_linear_velocity>0.95</max_linear_velocity>
+            <min_linear_velocity>-0.5</min_linear_velocity>
+            <max_linear_velocity>0.5</max_linear_velocity>
             <min_angular_velocity>-10.0</min_angular_velocity>
             <max_angular_velocity>10.0</max_angular_velocity>
-            <min_linear_acceleration>-5.0</min_linear_acceleration>
-            <max_linear_acceleration>3.0</max_linear_acceleration>
+            <min_linear_acceleration>-10.0</min_linear_acceleration>
+            <max_linear_acceleration>10.0</max_linear_acceleration>
             <min_angular_acceleration>-50.0</min_angular_acceleration>
             <max_angular_acceleration>50.0</max_angular_acceleration>

File: tuw_spike_description/model/spike/body/properties.xacro (robot description, xacro)
@@ -6,8 +6,8 @@
     <xacro:property name="wheel_z" value="-0.016"/>
     <xacro:property name="wheel_y" value="0.056"/>
-    <xacro:property name="wheel_diameter" value="0.056"/> <!-- lego diameter 56mm -->
+    <xacro:property name="wheel_diameter" value="0.056"/>
     <xacro:property name="wheel_radius" value="${wheel_diameter/2}"/>
-    <xacro:property name="wheel_len" value="0.0139"/> <!-- lego len 14mm -->
-    <xacro:property name="wheel_mass" value="0.016"/> <!-- kein gewicht von lego noch abwiegen-->
+    <xacro:property name="wheel_len" value="0.0139"/>
+    <xacro:property name="wheel_mass" value="0.016"/>
     <!-- Caster wheel from blender -->
     <xacro:property name="caster_z" value="-0.0344"/>
@@ -18,9 +18,8 @@
     <xacro:property name="caster_mass" value="0.005"/>
     <!-- base Chassis -->
-    <!-- Werte sind nur vorrübergehend -->
     <xacro:property name="chassis_mass" value="0.123"/>
     <xacro:property name="base_width" value="0.0879"/>
     <xacro:property name="base_length" value="0.170"/>
-    <xacro:property name="base_height" value="0.064"/>
+    <xacro:property name="base_height" value="0.008"/>
     <!-- from blender -->
     <xacro:property name="camera_x" value="0.099737"/>

File: tuw_spike_description/model/spike/body/wheels.xacro (robot description, xacro)
@@ -9,6 +9,4 @@
             <origin xyz="${wheel_x} ${y_reflect*wheel_y} ${wheel_z}" rpy="0 0 0" />
             <axis xyz="0 1 0"/>
-            <!-- <dynamics damping="0.2" />
-            <limit effort="100" velocity="3.0" /> -->
         </joint>
         <!-- Wheel Link -->
@@ -17,5 +15,5 @@
                 <origin xyz="0 0 0" rpy="${PI/2} 0 0" />
                 <geometry>
-                    <cylinder length="${wheel_len}" radius="${wheel_radius}" />
+                    <cylinder length="${wheel_len/10}" radius="${wheel_radius}" />
                 </geometry>
             </collision>

File: tuw_spike_description/model/spike/main.xacro (robot description, xacro)
@@ -1,17 +1,10 @@
 <?xml version="1.0"?>
 <robot xmlns:xacro="http://ros.org/wiki/xacro" name="spike" >
-  <xacro:arg name="models_dir"       default="model"/>
-  <xacro:arg name="robot_model"      default="spike"/>
-  <xacro:arg name="laser_model"      default="hokuyo"/>
   <xacro:arg name="namespace"        default="robot0"/>
-  <xacro:arg name="robot_name"       default="r0"/>
-  <xacro:property name="models_dir"    value="$(arg models_dir)"/>
   <xacro:property name="namespace"    value="$(arg namespace)"/>
-  <xacro:property name="robot_model"   value="$(arg robot_model)"/>
   <!-- Import Rviz colors -->
   <xacro:include filename="body/materials.xacro" />
   <!-- Import platform -->
   <xacro:include filename="body/body.xacro"/>
-  <!-- <xacro:vehicle_body name="body" parent="base_link"/> -->
   <!-- differential drive  and joint stage plugin -->
   <xacro:include filename="body/plugins.xacro"/>
