Commit message: moved simulation trajectory to analysis

File: tuw_spike_description/model/spike/body/wheels.xacro (robot description, xacro)
@@ -15,5 +15,5 @@
                 <origin xyz="0 0 0" rpy="${PI/2} 0 0" />
                 <geometry>
-                    <cylinder length="${wheel_len/10}" radius="${wheel_radius}" />
+                    <cylinder length="${wheel_len}" radius="${wheel_radius}" />
                 </geometry>
             </collision>
@@ -36,6 +36,6 @@
         </link>
         <gazebo reference="${prefix}_wheel">
-            <mu1 value="0.6"/>
-            <mu2 value="0.6"/>
+            <mu1 value="1.0"/>
+            <mu2 value="1.0"/>
             <fdir1 value="1 0 0"/>
         </gazebo>

File: tuw_spike_description/model/spike/main.xacro (robot description, xacro)
@@ -1,5 +1,5 @@
 <?xml version="1.0"?>
 <robot xmlns:xacro="http://ros.org/wiki/xacro" name="spike" >
-  <xacro:arg name="namespace"        default="robot0"/>
+  <xacro:arg name="namespace"        default=""/>
   <xacro:property name="namespace"    value="$(arg namespace)"/>
   <!-- Import Rviz colors -->
