Commit message: changed to wheel offset to new model

File: tuw_spike_description/model/spike/body/properties.xacro (robot description, xacro)
@@ -3,5 +3,5 @@
     <xacro:property name="PI" value="3.1415926535897931" />
     <!-- wheel from blender -->
-    <xacro:property name="wheel_x" value="-0.08"/>
+    <xacro:property name="wheel_x" value="-0.032"/>
     <xacro:property name="wheel_z" value="-0.016"/>
     <xacro:property name="wheel_y" value="0.056"/>
