Commit message: added new model

File: tuw_spike_description/model/spike/body/engine.xacro (robot description, xacro)
@@ -19,4 +19,11 @@
                     ixy="0.0" ixz="0.0" iyz="0.0" />
             </inertial>
+            <visual name="battery_visual">
+                <origin xyz="0 0 0" rpy="0 0 0" />
+                <geometry>
+                    <box size="${engine_length} ${engine_width} ${engine_height}" />
+                </geometry>
+                <material name="grey" />
+            </visual>
         </link>
     </xacro:macro>

File: tuw_spike_description/model/spike/body/properties.xacro (robot description, xacro)
@@ -35,7 +35,7 @@
     <xacro:property name="battery_length" value="0.071"/>
     <xacro:property name="battery_height" value="0.022"/>
-    <xacro:property name="battery_x" value="0.016"/>
+    <xacro:property name="battery_x" value="-0.040"/>
     <xacro:property name="battery_y" value="0.0"/>
-    <xacro:property name="battery_z" value="${-0.004 - (battery_height/2)}"/>
+    <xacro:property name="battery_z" value="${0.004 + (battery_height/2)}"/>
     <xacro:property name="battery_mass" value="0.150"/>
     <!-- from cad / blender -->
@@ -51,5 +51,5 @@
     <xacro:property name="engine_length" value="0.0715"/>
     <xacro:property name="engine_height" value="0.024"/>
-    <xacro:property name="engine_x" value="-0.056"/>
+    <xacro:property name="engine_x" value="-0.008"/>
     <xacro:property name="engine_y" value="0.032"/>
     <xacro:property name="engine_z" value="${-0.004 - engine_height/2}"/>
