Commit message: added wheel mesh, mesh paramter to spawn robot

File: tuw_spike_description/model/spike/body/chassis.xacro (robot description, xacro)
@@ -12,8 +12,11 @@
             <origin xyz="0 0 0" rpy="0 0 0" />
             <geometry>
-                <box size="${base_length} ${base_width} ${base_height}" />
-                 <!-- <mesh filename="package://tuw_spike_description/model/spike/body/mesh/model_chassis.dae"/> -->
+                <xacro:if value="${mesh_property}">
+                    <mesh filename="package://tuw_spike_description/model/spike/body/mesh/model_chassis.dae"/>
+                </xacro:if>
+                <xacro:unless value="${mesh_property}">
+                    <box size="${base_length} ${base_width} ${base_height}" />
+                </xacro:unless>
             </geometry>
-            <material name="orange" />
         </visual>
         <inertial name="base_link_inertia">

File: tuw_spike_description/model/spike/body/engine.xacro (robot description, xacro)
@@ -19,11 +19,13 @@
                     ixy="0.0" ixz="0.0" iyz="0.0" />
             </inertial>
-            <visual name="battery_visual">
-                <origin xyz="0 0 0" rpy="0 0 0" />
-                <geometry>
-                    <box size="${engine_length} ${engine_width} ${engine_height}" />
-                </geometry>
-                <material name="grey" />
-            </visual>
+            <xacro:unless value="${mesh_property}">
+                <visual name="battery_visual">
+                    <origin xyz="0 0 0" rpy="0 0 0" />
+                    <geometry>
+                        <box size="${engine_length} ${engine_width} ${engine_height}" />
+                    </geometry>
+                    <material name="grey" />
+                </visual>
+            </xacro:unless>
         </link>
     </xacro:macro>

File: tuw_spike_description/model/spike/body/pi.xacro (robot description, xacro)
@@ -14,5 +14,5 @@
                 <box size="${pi_length} ${pi_width} ${pi_height}" />
             </geometry>
-            <material name="grey" />
+            <material name="green" />
         </visual>
         <inertial name="pi_inertia">

File: tuw_spike_description/model/spike/body/wheels.xacro (robot description, xacro)
@@ -18,10 +18,20 @@
                 </geometry>
             </collision>
+            <xacro:if value="${mesh_property}">
+                <xacro:property name="wheel_rotation" value="0"/>
+            </xacro:if>
+            <xacro:unless value="${mesh_property}">
+                <xacro:property name="wheel_rotation" value="${PI/2}"/>
+            </xacro:unless>
             <visual>
-                <origin xyz="0 0 0" rpy="${PI/2} 0 0" />
+                <origin xyz="0 0 0" rpy="${wheel_rotation} 0 0" />
                 <geometry>
-                    <cylinder length="${wheel_len}" radius="${wheel_radius}" />
+                    <xacro:if value="${mesh_property}">
+                        <mesh filename="package://tuw_spike_description/model/spike/body/mesh/model_wheel.dae"/>
+                    </xacro:if>
+                    <xacro:unless value="${mesh_property}">
+                        <cylinder length="${wheel_len}" radius="${wheel_radius}" />
+                    </xacro:unless>
                 </geometry>
-                <material name="green" />
             </visual>
             <inertial>

File: tuw_spike_description/model/spike/main.xacro (robot description, xacro)
@@ -3,4 +3,6 @@
   <xacro:arg name="namespace"        default=""/>
   <xacro:property name="namespace"    value="$(arg namespace)"/>
+  <xacro:arg name="mesh" default="false"/>
+  <xacro:property name="mesh_property" value="$(arg mesh)"/>
   <!-- Import Rviz colors -->
   <xacro:include filename="body/materials.xacro" />
