Commit message: perform extrinsic calibration using checkerboard - set projection matrix equal to camera intrinsic matrix in calibration data - RectifyNode uses the projection matrix in initUndistorRectifyMap,   while undistort doesn't

File: tuw_spike_description/model/spike/body/camera.xacro (robot description, xacro)
@@ -29,5 +29,5 @@
     <link name="camera_optical"/>
     <joint name="camera_optical_joint" type="fixed">
-        <origin xyz="0 0 0" rpy="${-PI/2} 0 ${-PI/2}"/>
+        <origin xyz="0.0098 0.0015 -0.0017" rpy="-1.565 -0.018 -1.577"/>
         <parent link="camera"/>
         <child link="camera_optical"/>
